File: pcb/splitflappcb.kicad_pcb (KiCad board)
At the start: 2 copper layers, 302 x 25.4 mm, 43 parts, among them J1 Conn_01x04_Pin, J10 Conn_01x05_Pin, J11 HallSensor, J12 Conn_ARM_SWD_TagConnect_TC203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, J13 Conn_01x05_Pin, J14 HallSensor, J15 Conn_01x03_Pin, J16 Conn_01x05_Pin, J17 Conn_01x04_Pin, J2 HallSensor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

Commit message: S E N T
Parts:
- added C18: 100n, Capacitor_SMD:C_0603_1608Metric, F.Cu at (170.6, 29.0)
- added C19: 100n, Capacitor_SMD:C_0603_1608Metric, F.Cu at (164.4, 28.9)
- added R1: 20k, Resistor_SMD:R_0805_2012Metric, F.Cu at (39.0, 33.9)
- added R10: 20k, Resistor_SMD:R_0805_2012Metric, F.Cu at (185.1, 26.8)
- added R11: 20k, Resistor_SMD:R_0805_2012Metric, F.Cu at (240.6, 36.9)
- added R12: 20k, Resistor_SMD:R_0805_2012Metric, F.Cu at (290.9, 36.9)
- added R2: 20k, Resistor_SMD:R_0805_2012Metric, F.Cu at (89.3, 33.9)
- added R3: 20k, Resistor_SMD:R_0805_2012Metric, F.Cu at (139.8, 33.9)
- added R4: 20k, Resistor_SMD:R_0805_2012Metric, F.Cu at (187.1, 30.4)
- added R5: 20k, Resistor_SMD:R_0805_2012Metric, F.Cu at (240.6, 33.9)
- added R6: 20k, Resistor_SMD:R_0805_2012Metric, F.Cu at (290.9, 33.9)
- added R7: 20k, Resistor_SMD:R_0805_2012Metric, F.Cu at (39.0, 36.9)
- added R8: 20k, Resistor_SMD:R_0805_2012Metric, F.Cu at (89.3, 36.9)
- added R9: 20k, Resistor_SMD:R_0805_2012Metric, F.Cu at (139.8, 36.9)
- added U8: LDO, Package_TO_SOT_SMD:SOT-23-3, F.Cu at (167.5, 28.9)
- J15: value Conn_01x03_Pin -> ~; footprint Connector_PinHeader_2.54mm:PinHeader_1x03_P2.54mm_Vertical -> Package_TO_SOT_SMD:SOT-89-3
- moved C14 5.45 mm to (237.5, 26.9), turned to -90 degrees
- moved J15 3.52 mm to (274.7, 31.6)
Connections:
- C1 pad 1: +3V3 -> +5V
- C11 pad 1: +3V3 -> +5V
- C14 pad 1: +3V3 -> +5V
- C16 pad 1: +3V3 -> +5V
- C3 pad 1: +3V3 -> +5V
- C5 pad 1: +3V3 -> +5V
- J1 pad 4: +3V3 -> +5V
- J11 pad 1: +3V3 -> +5V
- J11 pad 3: /5_H -> Net-(J11-Pin_3)
- J14 pad 1: +3V3 -> +5V
- J14 pad 3: /6_H -> Net-(J14-Pin_3)
- J17 pad 4: +3V3 -> +5V
- J2 pad 1: +3V3 -> +5V
- J2 pad 3: /1_H -> Net-(J2-Pin_3)
- J5 pad 1: +3V3 -> +5V
- J5 pad 3: /2_H -> Net-(J5-Pin_3)
- J6 pad 1: +3V3 -> +5V
- J6 pad 3: /3_H -> Net-(J6-Pin_3)
- J8 pad 1: +3V3 -> +5V
- J8 pad 3: /4_H -> Net-(J8-Pin_3)
Routing:
- net +5V: track 0.00 -> 380.8 mm
- net +3V3: track 429.4 -> 147.4 mm, vias 0 -> 5
- net Net-(J11-Pin_3): track 0.00 -> 3.30 mm
- net Net-(J5-Pin_3): track 0.00 -> 3.30 mm
- net Net-(J2-Pin_3): track 0.00 -> 3.30 mm
- net Net-(J6-Pin_3): track 0.00 -> 3.30 mm
- net Net-(J14-Pin_3): track 0.00 -> 3.30 mm
- net Net-(J8-Pin_3): track 0.00 -> 2.74 mm
- net /6_1: track 129.2 -> 130.9 mm
- net /4_1: track 29.2 -> 31.0 mm
- net /1_H: track 140.7 -> 142.2 mm
- net /3_H: track 35.2 -> 36.8 mm
- net /2_H: track 86.7 -> 88.2 mm
- net /4_H: track 17.8 -> 16.4 mm
- net /6_H: track 128.8 -> 127.4 mm
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Other:
- board text added: "5v"
- board text removed: "3v3"
