File: pcb/splitflappcb.kicad_sch (KiCad schematic)
At the start: 13 parts, among them J1 Conn_01x04_Pin, J12 Conn_ARM_SWD_TagConnect_TC203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, J15 Conn_01x03_Pin, J17 Conn_01x04_Pin, J9 Conn_01x04_Pin, U4 STM32F030C8Tx

Commit message: S E N T
Parts:
- added C18, C19: 100n, Capacitor_SMD:C_0603_1608Metric, symbol Device:C_Small
- added U8: LDO, Package_TO_SOT_SMD:SOT-23-3, symbol Regulator_Linear:AMS1117
- J15: value Conn_01x03_Pin -> ~; footprint Connector_PinHeader_2.54mm:PinHeader_1x03_P2.54mm_Vertical -> Package_TO_SOT_SMD:SOT-89-3; LCSC (none) -> C351450
- J9: LCSC C721444 -> C6332197
Connections:
- net +3V3: now also C18.1, U8.2 (VO); no longer J1.4 (Pin_4), J17.4 (Pin_4)
- net GND: now also C18.2, C19.2, U8.1 (ADJ)
- new net +5V: C19.1, J1.4 (Pin_4), J17.4 (Pin_4), U8.3 (VI)

Commit message: ordered ol
Parts:
- U4: LCSC C23922 -> C62514
Changed lines of the file:
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@@
 			)
 		)
-		(property "LCSC" "C23922"
+		(property "LCSC" "C62514"
 			(at 68.58 102.87 0)
 			(effects
